File: flipdot.kicad_pcb (KiCad board)
At the start: 2 copper layers, 121.3 x 197.5 mm, 521 parts, among them J10 Conn_01x02_Pin, J13 Conn_01x02_Pin, J14 Conn_01x02_Pin, J15 Conn_01x02_Pin, J17 Conn_01x02_Pin, J18 Conn_01x02_Pin, J19 Conn_01x02_Pin, J2 Conn_01x02_Pin, J21 Conn_01x02_Pin, J22 Conn_01x02_Pin, J25 Conn_01x02_Pin, J26 Conn_01x02_Pin, J27 Conn_01x02_Pin, J29 Conn_01x02_Pin, J3 Conn_01x02_Pin, J30 Conn_01x02_Pin, J31 Conn_01x02_Pin, J33 Conn_01x02_Pin, J34 Conn_01x02_Pin, J37 Conn_01x02_Pin, J38 Conn_01x02_Pin, J39 Conn_01x02_Pin, J4 Conn_01x05_Pin, J41 Conn_01x02_Pin, J42 Conn_01x02_Pin, J43 Conn_01x02_Pin, J45 Conn_01x02_Pin, J46 Conn_01x02_Pin, J49 Conn_01x02_Pin, J5 Conn_01x02_Pin, J50 Conn_01x02_Pin, J51 Conn_01x02_Pin, J6 Conn_01x02_Pin, J8 Conn_01x05_Pin, J9 Conn_01x02_Pin, Q1 FDN338P, U104 74HC595, U113 74HC595, U118 Megain MG6208T3-33, U14 74HC595, U23 74HC595, U32 74HC595, U41 74HC595, U5 74HC595, U50 74HC595, U59 74HC595, U68 74HC595, U77 74HC595, U86 74HC595, U95 74HC595

Commit message: initial halfboard
Parts:
- removed C105, C120, C121, C124, C130, C145, C146, C149, C155, C170, C171, C174, C180, C195, C196, C199, C20, C205, C21, C220, C221, C224, C230, C24, C245, C246, C249, C255, C27, C270, C271, C274, C28, C280, C29, C295, C296, C299, C30, C305, C31, C320, C321, C324, C45, C46, C49, C5, C55, C70, C71, C74, C80, C95, C96, C99: 47u, Flipdot:CP_Elec_5x5.4_slim
- removed C116, C117, C118, C119, C141, C142, C143, C144, C16, C166, C167, C168, C169, C17, C18, C19, C191, C192, C193, C194, C216, C217, C218, C219, C241, C242, C243, C244, C266, C267, C268, C269, C291, C292, C293, C294, C316, C317, C318, C319, C41, C42, C43, C44, C66, C67, C68, C69, C91, C92, C93, C94: 10u, Capacitor_SMD:C_0805_2012Metric
- removed D1: Blue, LED_SMD:LED_0603_1608Metric
- removed F1: nSMD050-33V, Fuse:Fuse_1206_3216Metric
- removed H10, H12, H14, H16, H18, H2, H20, H22, H24, H26, H4, H6, H8: MountingHole, MountingHole:MountingHole_3.2mm_M3_DIN965
- removed J13, J15, J17, J19, J2, J22, J26, J27, J29, J3, J31, J33, J37, J39, J42, J43, J46, J49, J51, J6, J9: Conn_01x02_Pin, Connector_JST:JST_VH_B2P-VH_1x02_P3.96mm_Vertical
- removed J4, J8: Conn_01x05_Pin, Connector_JST:JST_ZH_B6B-ZR_1x06_P1.50mm_Vertical
- removed L101, L102, L103, L104, L13, L14, L15, L16, L21, L22, L23, L24, L29, L30, L31, L32, L37, L38, L39, L40, L45, L46, L47, L48, L5, L53, L54, L55, L56, L6, L61, L62, L63, L64, L69, L7, L70, L71, L72, L77, L78, L79, L8, L80, L85, L86, L87, L88, L93, L94, L95, L96: ~, Flipdot:Flipdot_single
- removed R2: 100K, Resistor_SMD:R_0603_1608Metric
- removed TP2: OUT, TestPoint:TestPoint_Pad_D1.5mm
- removed TP3: CLK, TestPoint:TestPoint_Pad_D1.5mm
- removed TP6: OE*, TestPoint:TestPoint_Pad_D1.5mm
- removed TP8: VCC, TestPoint:TestPoint_Pad_D1.5mm
- removed U105, U106, U107, U108, U114, U115, U116, U117, U15, U16, U17, U18, U24, U25, U26, U27, U33, U34, U35, U36, U42, U43, U44, U45, U51, U52, U53, U54, U6, U60, U61, U62, U63, U69, U7, U70, U71, U72, U78, U79, U8, U80, U81, U87, U88, U89, U9, U90, U96, U97, U98, U99: ~, Package_SO:SOP-8_3.9x4.9mm_P1.27mm
- moved H1 2.83 mm to (1.20, -5.20)
- moved U118 0.99 mm to (55.7, 25.7)
Routing:
- net +12V: track 3897.2 -> 1268.6 mm, vias 275 -> 123
- net LATCH: track 1395.1 -> 735.2 mm
- net /row13/DATA_OUT: track 262.2 -> 0.00 mm
- net GND: track 732.4 -> 477.8 mm, vias 521 -> 290
- net CLK: track 349.7 -> 265.4 mm, vias 27 -> 25
- net OE*: track 325.1 -> 251.6 mm, vias 25 -> 26
- net VCC: track 469.7 -> 400.6 mm, vias 24 -> 25
- net Net-(U68-QA): track 51.9 -> 0.00 mm, vias 2 -> 0
- net Net-(U95-QA): track 51.9 -> 0.00 mm, vias 2 -> 0
- net Net-(U23-QA): track 51.9 -> 0.00 mm, vias 2 -> 0
- net Net-(U86-QA): track 51.9 -> 0.00 mm, vias 2 -> 0
- net Net-(U77-QA): track 51.9 -> 0.00 mm, vias 2 -> 0
- net Net-(U50-QA): track 51.9 -> 0.00 mm, vias 2 -> 0
- net Net-(U41-QA): track 51.9 -> 0.00 mm, vias 2 -> 0
- net Net-(U32-QA): track 51.9 -> 0.00 mm, vias 2 -> 0
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Other:
- board size 121.3 x 197.5 mm -> 60.4 x 197.5 mm
- board text added: "2026-06-04"
- board text removed: "2026-05-18"
- board text removed: "Plywood frame"
- board text removed: "big electrolytics"

Commit message: add 12v caps back in
Parts:
- removed H11, H15, H23, H3: MountingHole, MountingHole:MountingHole_3.2mm_M3_DIN965
- removed J21, J30, J45, J5: Conn_01x02_Pin, Connector_JST:JST_VH_B2P-VH_1x02_P3.96mm_Vertical
- added C27: 47u, Flipdot:CP_Elec_5x5.4_slim, F.Cu at (8.60, 13.4)
- added C28: 47u, Flipdot:CP_Elec_5x5.4_slim, F.Cu at (8.70, 74.2)
- added C29: 47u, Flipdot:CP_Elec_5x5.4_slim, F.Cu at (8.70, 104.8)
- added C31: 47u, Flipdot:CP_Elec_5x5.4_slim, F.Cu at (8.70, 165.8)
Routing:
- net GND: track 477.8 -> 463.4 mm, vias 290 -> 305
- net +12V: track 1268.6 -> 1259.4 mm
