File: flipdot-decode.kicad_sch (KiCad schematic)
At the start: 8 parts, among them J1 Conn_01x05_Pin, J2 Conn_01x06_Pin, SW1 SW_DIP_x05, U1 CH32V003FxUx, U2 MAX485E

Commit message: board designed
Parts:
- removed U1: CH32V003FxUx, Package_DFN_QFN:QFN-20-1EP_3x3mm_P0.4mm_EP1.65x1.65mm, symbol MCU_WCH_CH32V0:CH32V003FxUx
- added C2: 0.1u, Capacitor_SMD:C_0603_1608Metric, symbol Device:C_Small
- added J3: Conn_01x03_Pin, Connector_PinHeader_2.54mm:PinHeader_1x03_P2.54mm_Vertical, symbol Connector:Conn_01x03_Pin
- added U3: CH32V003FxPx, Package_SO:TSSOP-20_4.4x6.5mm_P0.65mm, symbol MCU_WCH_RiscV:CH32V003FxPx
- C1: value C_Small -> 0.1u
Connections:
- net VDD is gone; now on net VCC: C1.1
- net CLK: now also U3.15 (PC5)
- net DATA: now also U3.16 (PC6)
- net GND: now also C2.2, J3.2 (Pin_2), U3.7 (VSS)
- net OE*: now also U3.12 (PC2)
- net UART: now also U3.3 (PD6)
- net VBAT: now also U3.5 (PA1)
- net VCC: now also C2.1, J3.1 (Pin_1), U3.9 (VDD)
- net at SW1.2: now also U3.19 (PD2)
- net at SW1.3: now also U3.20 (PD3)
- net at SW1.4: now also U3.1 (PD4)
- net at SW1.5: now also U3.2 (PD5)
- net at SW1.1: now also U3.8 (PD0)
- new net NRST: U3.4 (PD7)
- new net SWD: J3.3 (Pin_3), U3.18 (PD1)
Other:
- moved on the sheet: C1, SW1

Commit message: add reset pin
Parts:
- J3: value Conn_01x03_Pin -> Conn_01x04_Pin; footprint Connector_PinHeader_2.54mm:PinHeader_1x03_P2.54mm_Vertical -> Connector_PinHeader_2.54mm:PinHeader_1x04_P2.54mm_Vertical; symbol Connector:Conn_01x03_Pin -> Connector:Conn_01x04_Pin
- R1: value R_Small -> 470K
- R2: value R_Small -> 150K
Connections:
- net GND: now also J3.3 (Pin_3); no longer J3.2 (Pin_2)
- net NRST: now also J3.1 (Pin_1)
- net SWD: now also J3.4 (Pin_4); no longer J3.3 (Pin_3)
- net VCC: now also J3.2 (Pin_2); no longer J3.1 (Pin_1)
Other:
- note added: "150/(470+150) = 0.242 Lipo max 12.6V => 3.048V Lipo min 9V => 2.177V DC supply 14V => 3.387V"
Changed lines of the file:
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@@
 	(generator_version "10.0")
 	(paper "A3")
+	(text "150/(470+150) = 0.242\nLipo max 12.6V => 3.048V\nLipo min 9V => 2.177V\nDC supply 14V => 3.387V"
+		(exclude_from_sim no)
+		(at 57.404 122.682 0)
+		(effects
+			(font
+				(size 1.27 1.27)
+			)
+			(justify left)
+		)
+	)
 	(text "euroknob uses PA1"
 		(exclude_from_sim no)
@@
 	(wire
 		(pts
+			(xy 137.16 132.08) (xy 152.4 132.08)
+		)
+		(stroke
+			(width 0)
+			(type default)
+		)
+	)
+	(wire
+		(pts
 			(xy 129.54 109.22) (xy 129.54 114.3)
 		)
@@
 			)
 			(justify left bottom)
+		)
+	)
+	(label "NRST"
+		(at 152.4 132.08 180)
+		(effects
+			(font
+				(size 1.27 1.27)
+			)
+			(justify right bottom)
 		)
 	)
@@
 			)
 		)
-		(property "Value" "R_Small"
+		(property "Value" "470K"
 			(at 46.99 105.4099 0)
 			(show_name no)
@@
 			)
 		)
-		(property "Value" "R_Small"
+		(property "Value" "150K"
 			(at 46.99 115.5699 0)
 			(show_name no)
@@
 	)
 	(symbol
-		(lib_id "Connector:Conn_01x03_Pin")
-		(at 132.08 137.16 0)
+		(lib_id "Connector:Conn_01x04_Pin")
+		(at 132.08 134.62 0)
 		(unit 1)
 		(body_style 1)
@@
 		(fields_autoplaced yes)
 		(property "Reference" "J3"
+			(at 132.715 127 0)
+			(show_name no)
+			(do_not_autoplace no)
+			(effects
+				(font
+					(size 1.27 1.27)
+				)
+			)
+		)
+		(property "Value" "Conn_01x04_Pin"
 			(at 132.715 129.54 0)
 			(show_name no)
@@
 			)
 		)
-		(property "Value" "Conn_01x03_Pin"
-			(at 132.715 132.08 0)
-			(show_name no)
-			(do_not_autoplace no)
-			(effects
-				(font
-					(size 1.27 1.27)
-				)
-			)
-		)
-		(property "Footprint" "Connector_PinHeader_2.54mm:PinHeader_1x03_P2.54mm_Vertical"
-			(at 132.08 137.16 0)
+		(property "Footprint" "Connector_PinHeader_2.54mm:PinHeader_1x04_P2.54mm_Vertical"
+			(at 132.08 134.62 0)
 			(hide yes)
 			(show_name no)
@@
 		)
 		(property "Datasheet" ""
-			(at 132.08 137.16 0)
-			(hide yes)
-			(show_name no)
-			(do_not_autoplace no)
-			(effects
-				(font
-					(size 1.27 1.27)
-				)
-			)
-		)
-		(property "Description" "Generic connector, single row, 01x03, script generated"
-			(at 132.08 137.16 0)
+			(at 132.08 134.62 0)
+			(hide yes)
+			(show_name no)
+			(do_not_autoplace no)
+			(effects
+				(font
+					(size 1.27 1.27)
+				)
+			)
+		)
+		(property "Description" "Generic connector, single row, 01x04, script generated"
+			(at 132.08 134.62 0)
 			(hide yes)
 			(show_name no)
@@
 		(pin "1"
 		)
+		(pin "4"
+		)
 		(instances
